File: Board/AriaBoard.sch (KiCad schematic (older format))
At the start: 34 parts, among them J1 USB_MICRO, J2 HR911105_RJ45, P1 CONN_2, P10 CONN_9, P11 CONN_4, P12 CONN_4, P13 CONN_4, P14 CONN_4, P2 CONN_2, P3 CONN_4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

Commit message: routing in progress
Parts:
- removed R1: 0, ~, symbol R
Connections:
- net labels removed: AGND
- wire segments 45 -> 44
Changed lines of the file:
@@
 Sheet 1 4
 Title "AriaBoard"
-Date "25 mar 2015"
+Date "14 apr 2015"
 Rev "0.1"
 Comp "Associazione Pometeo"
@@
 $EndComp
 $Comp
-L AGND #PWR01
-U 1 1 55132B34
-P 750 1450
-F 0 "#PWR01" H 750 1450 40  0001 C CNN
-F 1 "AGND" H 750 1380 50  0000 C CNN
-F 2 "~" H 750 1450 60  0000 C CNN
-F 3 "~" H 750 1450 60  0000 C CNN
-	1    750  1450
-	1    0    0    -1
-$EndComp
-$Comp
-L DGND #PWR02
+L DGND #PWR01
 U 1 1 55132B43
 P 1250 1450
-F 0 "#PWR02" H 1250 1450 40  0001 C CNN
+F 0 "#PWR01" H 1250 1450 40  0001 C CNN
 F 1 "DGND" H 1250 1380 40  0000 C CNN
 F 2 "~" H 1250 1450 60  0000 C CNN
@@
 $EndComp
 $Comp
-L PGND #PWR03
+L PGND #PWR02
 U 1 1 55132C06
 P 1850 1450
-F 0 "#PWR03" H 1850 1450 40  0001 C CNN
+F 0 "#PWR02" H 1850 1450 40  0001 C CNN
 F 1 "PGND" H 1850 1380 40  0000 C CNN
 F 2 "~" H 1850 1450 60  0000 C CNN
@@
 $EndComp
 $Comp
-L R R1
-U 1 1 55132C70
-P 1000 1250
-F 0 "R1" V 1080 1250 40  0000 C CNN
-F 1 "0" V 1007 1251 40  0000 C CNN
-F 2 "~" V 930 1250 30  0000 C CNN
-F 3 "~" H 1000 1250 30  0000 C CNN
-	1    1000 1250
-	0    -1   -1   0
-$EndComp
-$Comp
-L PWR_FLAG #FLG04
+L PWR_FLAG #FLG03
 U 1 1 55132DF3
 P 1250 1250
-F 0 "#FLG04" H 1250 1345 30  0001 C CNN
+F 0 "#FLG03" H 1250 1345 30  0001 C CNN
 F 1 "PWR_FLAG" H 1250 1430 30  0000 C CNN
 F 2 "~" H 1250 1250 60  0000 C CNN
@@
 $EndComp
 $Comp
-L PWR_FLAG #FLG05
-U 1 1 55132E00
-P 750 1250
-F 0 "#FLG05" H 750 1345 30  0001 C CNN
-F 1 "PWR_FLAG" H 750 1430 30  0000 C CNN
-F 2 "~" H 750 1250 60  0000 C CNN
-F 3 "~" H 750 1250 60  0000 C CNN
-	1    750  1250
-	1    0    0    -1
-$EndComp
-$Comp
-L PWR_FLAG #FLG06
+L PWR_FLAG #FLG04
 U 1 1 55132E06
 P 1850 1250
-F 0 "#FLG06" H 1850 1345 30  0001 C CNN
+F 0 "#FLG04" H 1850 1345 30  0001 C CNN
 F 1 "PWR_FLAG" H 1850 1430 30  0000 C CNN
 F 2 "~" H 1850 1250 60  0000 C CNN
@@
 3v_reg_vcc
 $Comp
-L PWR_FLAG #FLG07
+L PWR_FLAG #FLG05
 U 1 1 5513680B
 P 5350 1000
-F 0 "#FLG07" H 5350 1095 30  0001 C CNN
+F 0 "#FLG05" H 5350 1095 30  0001 C CNN
 F 1 "PWR_FLAG" H 5350 1180 30  0000 C CNN
 F 2 "~" H 5350 1000 60  0000 C CNN
@@
 $EndComp
 $Comp
-L PWR_FLAG #FLG08
+L PWR_FLAG #FLG06
 U 1 1 55136818
 P 4750 1000
-F 0 "#FLG08" H 4750 1095 30  0001 C CNN
+F 0 "#FLG06" H 4750 1095 30  0001 C CNN
 F 1 "PWR_FLAG" H 4750 1180 30  0000 C CNN
 F 2 "~" H 4750 1000 60  0000 C CNN
@@
 $EndComp
 $Comp
-L PWR_FLAG #FLG09
+L PWR_FLAG #FLG07
 U 1 1 5513681E
 P 4150 1000
-F 0 "#FLG09" H 4150 1095 30  0001 C CNN
+F 0 "#FLG07" H 4150 1095 30  0001 C CNN
 F 1 "PWR_FLAG" H 4150 1180 30  0000 C CNN
 F 2 "~" H 4150 1000 60  0000 C CNN
@@
 $EndComp
 $Comp
-L VCC #PWR010
+L VCC #PWR08
 U 1 1 55136A6F
 P 4850 1000
-F 0 "#PWR010" H 4850 1100 30  0001 C CNN
+F 0 "#PWR08" H 4850 1100 30  0001 C CNN
 F 1 "VCC" H 4850 1100 30  0000 C CNN
 F 2 "~" H 4850 1000 60  0000 C CNN
@@
 $EndComp
 $Comp
-L PGND #PWR011
+L PGND #PWR09
 U 1 1 55137C99
 P 1000 3825
-F 0 "#PWR011" H 1000 3825 40  0001 C CNN
+F 0 "#PWR09" H 1000 3825 40  0001 C CNN
 F 1 "PGND" H 1000 3755 40  0000 C CNN
 F 2 "~" H 1000 3825 60  0000 C CNN
@@
 5v_reg_vcc
 $Comp
-L DGND #PWR012
+L DGND #PWR010
 U 1 1 5513BE77
 P 14200 4500
-F 0 "#PWR012" H 14200 4500 40  0001 C CNN
+F 0 "#PWR010" H 14200 4500 40  0001 C CNN
 F 1 "DGND" H 14200 4430 40  0000 C CNN
 F 2 "~" H 14200 4500 60  0000 C CNN
@@
 $EndComp
 $Comp
-L DGND #PWR013
+L DGND #PWR011
 U 1 1 5513BF15
 P 14650 5050
-F 0 "#PWR013" H 14650 5050 40  0001 C CNN
+F 0 "#PWR011" H 14650 5050 40  0001 C CNN
 F 1 "DGND" H 14650 4980 40  0000 C CNN
 F 2 "~" H 14650 5050 60  0000 C CNN
@@
 $EndComp
 $Comp
-L DGND #PWR014
+L DGND #PWR012
 U 1 1 5513CD91
 P 10450 7925
-F 0 "#PWR014" H 10450 7925 40  0001 C CNN
+F 0 "#PWR012" H 10450 7925 40  0001 C CNN
 F 1 "DGND" H 10450 7855 40  0000 C CNN
 F 2 "~" H 10450 7925 60  0000 C CNN
@@
 $EndComp
 $Comp
-L DGND #PWR015
+L DGND #PWR013
 U 1 1 5513D0FF
 P 10950 8475
-F 0 "#PWR015" H 10950 8475 40  0001 C CNN
+F 0 "#PWR013" H 10950 8475 40  0001 C CNN
 F 1 "DGND" H 10950 8405 40  0000 C CNN
 F 2 "~" H 10950 8475 60  0000 C CNN
@@
 $EndComp
 $Comp
-L PGND #PWR016
+L PGND #PWR014
 U 1 1 5513D2C9
 P 14300 9800
-F 0 "#PWR016" H 14300 9800 40  0001 C CNN
+F 0 "#PWR014" H 14300 9800 40  0001 C CNN
 F 1 "PGND" H 14300 9730 40  0000 C CNN
 F 2 "~" H 14300 9800 60  0000 C CNN
@@
 $EndComp
 $Comp
-L PGND #PWR017
+L PGND #PWR015
 U 1 1 5513D2E0
 P 13050 9800
-F 0 "#PWR017" H 13050 9800 40  0001 C CNN
+F 0 "#PWR015" H 13050 9800 40  0001 C CNN
 F 1 "PGND" H 13050 9730 40  0000 C CNN
 F 2 "~" H 13050 9800 60  0000 C CNN
@@
 $EndComp
 $Comp
-L PGND #PWR018
+L PGND #PWR016
 U 1 1 5513D313
 P 13700 9800
-F 0 "#PWR018" H 13700 9800 40  0001 C CNN
+F 0 "#PWR016" H 13700 9800 40  0001 C CNN
 F 1 "PGND" H 13700 9730 40  0000 C CNN
 F 2 "~" H 13700 9800 60  0000 C CNN
@@
 $EndComp
 $Comp
-L PGND #PWR019
+L PGND #PWR017
 U 1 1 5513DE4C
 P 9825 9600
-F 0 "#PWR019" H 9825 9600 40  0001 C CNN
+F 0 "#PWR017" H 9825 9600 40  0001 C CNN
 F 1 "PGND" H 9825 9530 40  0000 C CNN
 F 2 "~" H 9825 9600 60  0000 C CNN
@@
 $EndComp
 $Comp
-L DGND #PWR020
+L DGND #PWR018
 U 1 1 5513DFF0
 P 8825 9950
-F 0 "#PWR020" H 8825 9950 40  0001 C CNN
+F 0 "#PWR018" H 8825 9950 40  0001 C CNN
 F 1 "DGND" H 8825 9880 40  0000 C CNN
 F 2 "~" H 8825 9950 60  0000 C CNN
@@
 $EndComp
 $Comp
-L +5V #PWR021
+L +5V #PWR019
 U 1 1 5513E42A
 P 1000 2025
-F 0 "#PWR021" H 1000 2115 20  0001 C CNN
+F 0 "#PWR019" H 1000 2115 20  0001 C CNN
 F 1 "+5V" H 1000 2115 30  0000 C CNN
 F 2 "~" H 1000 2025 60  0000 C CNN
@@
 $EndComp
 $Comp
-L PWR_FLAG #FLG022
+L PWR_FLAG #FLG020
 U 1 1 5513E5F5
 P 1000 2200
-F 0 "#FLG022" H 1000 2295 30  0001 C CNN
+F 0 "#FLG020" H 1000 2295 30  0001 C CNN
 F 1 "PWR_FLAG" H 1000 2380 30  0000 C CNN
 F 2 "~" H 1000 2200 60  0000 C CNN
@@
 5v_usb
 $Comp
-L PWR_FLAG #FLG023
+L PWR_FLAG #FLG021
 U 1 1 5513EB2B
 P 1500 2025
-F 0 "#FLG023" H 1500 2120 30  0001 C CNN
+F 0 "#FLG021" H 1500 2120 30  0001 C CNN
 F 1 "PWR_FLAG" H 1500 2205 30  0000 C CNN
 F 2 "~" H 1500 2025 60  0000 C CNN
@@
 $EndComp
 $Comp
-L PWR_FLAG #FLG024
+L PWR_FLAG #FLG022
 U 1 1 5513EB38
 P 1500 2200
-F 0 "#FLG024" H 1500 2295 30  0001 C CNN
+F 0 "#FLG022" H 1500 2295 30  0001 C CNN
 F 1 "PWR_FLAG" H 1500 2380 30  0000 C CNN
 F 2 "~" H 1500 2200 60  0000 C CNN
@@
 Wire Wire Line
 	8300 10025 8300 9650
-Wire Wire Line
-	750  1450 750  1250
 Wire Wire Line
 	1250 1450 1250 1250
@@
 $EndComp
 $Comp
-L PWR_FLAG #FLG025
+L PWR_FLAG #FLG023
 U 1 1 5513EF13
 P 2825 2300
-F 0 "#FLG025" H 2825 2395 30  0001 C CNN
+F 0 "#FLG023" H 2825 2395 30  0001 C CNN
 F 1 "PWR_FLAG" H 2825 2480 30  0000 C CNN
 F 2 "~" H 2825 2300 60  0000 C CNN
@@
 3v_ftdi
 $Comp
-L PWR_FLAG #FLG026
+L PWR_FLAG #FLG024
 U 1 1 5513EF1B
 P 3325 2125
-F 0 "#FLG026" H 3325 2220 30  0001 C CNN
+F 0 "#FLG024" H 3325 2220 30  0001 C CNN
 F 1 "PWR_FLAG" H 3325 2305 30  0000 C CNN
 F 2 "~" H 3325 2125 60  0000 C CNN
@@
 $EndComp
 $Comp
-L PWR_FLAG #FLG027
+L PWR_FLAG #FLG025
 U 1 1 5513EF21
 P 3325 2300
-F 0 "#FLG027" H 3325 2395 30  0001 C CNN
+F 0 "#FLG025" H 3325 2395 30  0001 C CNN
 F 1 "PWR_FLAG" H 3325 2480 30  0000 C CNN
 F 2 "~" H 3325 2300 60  0000 C CNN
@@
 3v_ext
 $Comp
-L PWR_FLAG #FLG028
+L PWR_FLAG #FLG026
 U 1 1 5513F114
 P 3325 1875
-F 0 "#FLG028" H 3325 1970 30  0001 C CNN
+F 0 "#FLG026" H 3325 1970 30  0001 C CNN
 F 1 "PWR_FLAG" H 3325 2055 30  0000 C CNN
 F 2 "~" H 3325 1875 60  0000 C CNN
@@
 Connection ~ 2825 2125
 $Comp
-L PGND #PWR029
+L PGND #PWR027
 U 1 1 551493E7
 P 2850 3925
-F 0 "#PWR029" H 2850 3925 40  0001 C CNN
+F 0 "#PWR027" H 2850 3925 40  0001 C CNN
 F 1 "PGND" H 2850 3855 40  0000 C CNN
 F 2 "~" H 2850 3925 60  0000 C CNN
@@
 Grounds, Power Switch, Power Jumper and balance resistors
 $Comp
-L PGND #PWR030
+L PGND #PWR028
 U 1 1 5514AE44
 P 5025 10100
-F 0 "#PWR030" H 5025 10100 40  0001 C CNN
+F 0 "#PWR028" H 5025 10100 40  0001 C CNN
 F 1 "PGND" H 5025 10030 40  0000 C CNN
 F 2 "~" H 5025 10100 60  0000 C CNN
@@
 $EndComp
 $Comp
-L PGND #PWR031
+L PGND #PWR029
 U 1 1 5514AEAB
 P 6075 10850
-F 0 "#PWR031" H 6075 10850 40  0001 C CNN
+F 0 "#PWR029" H 6075 10850 40  0001 C CNN
 F 1 "PGND" H 6075 10780 40  0000 C CNN
 F 2 "~" H 6075 10850 60  0000 C CNN
@@
 3v_aria
 $Comp
-L PGND #PWR032
+L PGND #PWR030
 U 1 1 5514D3AC
 P 14650 6675
-F 0 "#PWR032" H 14650 6675 40  0001 C CNN
+F 0 "#PWR030" H 14650 6675 40  0001 C CNN
 F 1 "PGND" H 14650 6605 40  0000 C CNN
 F 2 "~" H 14650 6675 60  0000 C CNN
@@
 $EndComp
 $Comp
-L PGND #PWR033
+L PGND #PWR031
 U 1 1 5514D3B9
 P 14650 7050
-F 0 "#PWR033" H 14650 7050 40  0001 C CNN
+F 0 "#PWR031" H 14650 7050 40  0001 C CNN
 F 1 "PGND" H 14650 6980 40  0000 C CNN
 F 2 "~" H 14650 7050 60  0000 C CNN
@@
 3v_ext
 $Comp
-L PGND #PWR034
+L PGND #PWR032
 U 1 1 5514E6C7
 P 9725 2100
-F 0 "#PWR034" H 9725 2100 40  0001 C CNN
+F 0 "#PWR032" H 9725 2100 40  0001 C CNN
 F 1 "PGND" H 9725 2030 40  0000 C CNN
 F 2 "~" H 9725 2100 60  0000 C CNN
@@
 3v_ext
 $Comp
-L PGND #PWR035
+L PGND #PWR033
 U 1 1 55130463
 P 15625 8250
-F 0 "#PWR035" H 15625 8250 40  0001 C CNN
+F 0 "#PWR033" H 15625 8250 40  0001 C CNN
 F 1 "PGND" H 15625 8180 40  0000 C CNN
 F 2 "~" H 15625 8250 60  0000 C CNN
@@
 $EndComp
 $Comp
-L PGND #PWR036
+L PGND #PWR034
 U 1 1 551314BB
 P 15175 9750
-F 0 "#PWR036" H 15175 9750 40  0001 C CNN
+F 0 "#PWR034" H 15175 9750 40  0001 C CNN
 F 1 "PGND" H 15175 9680 40  0000 C CNN
 F 2 "~" H 15175 9750 60  0000 C CNN
